File: hardware/sousvide.kicad_pcb (KiCad board)
At the start: 2 copper layers, 100 x 75 mm, 66 parts, among them CON101 AVR-ISP-6, IC101 ATMEGA8-P, P101 CONN_01X06, P102 CONN_01X03, P103 CONN_01X03, P104 CONN_01X03, P105 CONN_01X08, P106 CONN_01X08, T101 TRANSFO, U101 TRIAC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

Commit message: Added Licensing information and authors file
Routing:
- net (no net): track 0.00 -> 15.8 mm
- net GND: track 116.6 -> 100.8 mm
Changed lines of the file:
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@@
-(kicad_pcb (version 4) (host pcbnew "(2016-04-29 BZR 6716)-stable")
+(kicad_pcb (version 20160815) (host pcbnew "(2016-12-18 revision 3ffa37c8b)-master")
   (general
     (links 122)
     (no_connects 0)
-    (area 170.5 11.1625 283.9925 93.245001)
+    (area 163.5 18.6625 276.9925 100.745001)
     (thickness 1.6)
     (drawings 9)
@@
   (page A4)
   (title_block
-    (title "Sous-Vide Temperature Controler")
+    (title "Sous-Vide Temperature Controller")
     (date 2016-08-03)
     (rev 1)
-    (company dynamic-noise.net)
-    (comment 1 "Gregor Vollmer")
+    (company "Gregor Vollmer <git@dynamic-noise.net>")
+    (comment 1 "(c) 2016 GPLv3")
   )
   (layers
@@
   )
   (setup
-    (last_trace_width 0.8)
+    (last_trace_width 0.25)
     (user_trace_width 0.3)
     (user_trace_width 0.4)
@@
     (uvia_dia 0.3)
     (uvia_drill 0.1)
+    (diff_pair_gap 0.25)
+    (diff_pair_width 0.2)
     (add_net +5V)
     (add_net /!RESET)
@@
     (uvia_dia 0.3)
     (uvia_drill 0.1)
+    (diff_pair_gap 0.25)
+    (diff_pair_width 0.2)
     (add_net /Live)
     (add_net Earth)
@@
     (arrow2b (pts (xy 171.5 20.5) (xy 172.086421 21.626504)))
   )
+  (segment (start 242.5 66.074188) (end 244.168523 67.742711) (width 0.25) (layer B.Cu) (net 0))
+  (segment (start 242.805329 57.593624) (end 242.805329 59.633667) (width 0.25) (layer B.Cu) (net 0))
+  (segment (start 242.805329 59.633667) (end 242.5 59.938996) (width 0.25) (layer B.Cu) (net 0))
+  (segment (start 242.5 59.938996) (end 242.5 66.074188) (width 0.25) (layer B.Cu) (net 0))
+  (segment (start 244.168523 67.742711) (end 248.742711 67.742711) (width 0.25) (layer B.Cu) (net 0))
+  (segment (start 248.742711 67.742711) (end 248.91499 67.91499) (width 0.25) (layer B.Cu) (net 0))
   (segment (start 209 32) (end 209 36.903792) (width 2.5) (layer B.Cu) (net 1))
   (segment (start 209 36.903792) (end 209.048104 36.951896) (width 2.5) (layer B.Cu) (net 1))
@@
   (segment (start 225.5 80.5) (end 225.5 83.5) (width 0.8) (layer B.Cu) (net 3))
   (segment (start 251.238686 56.46) (end 250.105062 57.593624) (width 0.25) (layer B.Cu) (net 4))
-  (segment (start 242.5 66.074188) (end 244.168523 67.742711) (width 0.25) (layer B.Cu) (net 4))
-  (segment (start 242.805329 57.593624) (end 242.805329 59.633667) (width 0.25) (layer B.Cu) (net 4))
-  (segment (start 242.805329 59.633667) (end 242.5 59.938996) (width 0.25) (layer B.Cu) (net 4))
-  (segment (start 242.5 59.938996) (end 242.5 66.074188) (width 0.25) (layer B.Cu) (net 4))
-  (segment (start 244.168523 67.742711) (end 248.742711 67.742711) (width 0.25) (layer B.Cu) (net 4))
-  (segment (start 248.742711 67.742711) (end 248.91499 67.91499) (width 0.25) (layer B.Cu) (net 4))
   (segment (start 244.5 84) (end 244.5 76.75) (width 0.25) (layer F.Cu) (net 4))
   (via (at 244.5 76.75) (size 1.2) (drill 0.8) (layers F.Cu B.Cu) (net 4))
